File: kicad/adaesc.kicad_pcb (KiCad board)
At the start: 2 copper layers, 10 parts

Commit message: traces
Routing:
- net (no net): track 0.62 -> 519.5 mm

Commit message: uhh
Parts:
- added REF**: square, square library:square, F.Cu at (90.5, 47.5)
- added REF**: square, square library:square, F.Cu at (101.0, 47.5)
Routing:
- net (no net): track 519.5 -> 705.2 mm, vias 0 -> 2

Commit message: whug
Routing:
- net (no net): track 705.2 -> 739.6 mm, vias 2 -> 8
Changed lines of the file:
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@@
+	)
+	(segment
+		(start 36.5 101.75)
+		(end 36.25 101.75)
+		(width 0.2)
+		(layer "F.Cu")
+		(net 0)
 	)
 	(segment
@@
 	(segment
 		(start 41.5 101.75)
-		(end 36.25 101.75)
+		(end 36.5 101.75)
 		(width 0.2)
 		(layer "F.Cu")
@@
 	)
 	(via
+		(at 57.92 101.5)
+		(size 0.6)
+		(drill 0.3)
+		(layers "F.Cu" "B.Cu")
+		(net 0)
+	)
+	(via
+		(at 79.96 102)
+		(size 0.6)
+		(drill 0.3)
+		(layers "F.Cu" "B.Cu")
+		(net 0)
+	)
+	(via
+		(at 81.46 73.95)
+		(size 0.6)
+		(drill 0.3)
+		(layers "F.Cu" "B.Cu")
+		(net 0)
+	)
+	(via
+		(at 36.5 101.75)
+		(size 0.6)
+		(drill 0.3)
+		(layers "F.Cu" "B.Cu")
+		(net 0)
+	)
+	(via
+		(at 59.5 73.95)
+		(size 0.6)
+		(drill 0.3)
+		(layers "F.Cu" "B.Cu")
+		(net 0)
+	)
+	(via
 		(at 90 51.5)
 		(size 0.6)
@@
 	)
 	(via
+		(at 35.42 74)
+		(size 0.6)
+		(drill 0.3)
+		(layers "F.Cu" "B.Cu")
+		(net 0)
+	)
+	(via
 		(at 100 51.5)
 		(size 0.6)
@@
 	)
 	(segment
-		(start 36.42 101.75)
-		(end 57.92 101.75)
+		(start 57.92 97.92)
+		(end 57.5 97.5)
+		(width 0.2)
+		(layer "B.Cu")
+		(net 0)
+	)
+	(segment
+		(start 81.5 97.5)
+		(end 82.5 96.5)
+		(width 0.2)
+		(layer "B.Cu")
+		(net 0)
+	)
+	(segment
+		(start 57.5 97.5)
+		(end 80 97.5)
+		(width 0.2)
+		(layer "B.Cu")
+		(net 0)
+	)
+	(segment
+		(start 57.92 101.5)
+		(end 57.92 97.92)
+		(width 0.2)
+		(layer "B.Cu")
+		(net 0)
+	)
+	(segment
+		(start 99 52.5)
+		(end 99.575736 51.924264)
 		(width 0.2)
 		(layer "B.Cu")
@@
 	(segment
 		(start 81.46 73.95)
-		(end 59.47 73.95)
+		(end 59.5 73.95)
+		(width 0.2)
+		(layer "B.Cu")
+		(net 0)
+	)
+	(segment
+		(start 99 96.5)
+		(end 99 52.5)
 		(width 0.2)
 		(layer "B.Cu")
@@
 	)
 	(segment
-		(start 79.96 102.2)
-		(end 79.96 76.04)
-		(width 0.2)
-		(layer "B.Cu")
-		(net 0)
-	)
-	(segment
 		(start 59.47 73.95)
 		(end 59.42 74)
@@
 	)
 	(segment
-		(start 80 76)
-		(end 81 76)
-		(width 0.2)
-		(layer "B.Cu")
-		(net 0)
-	)
-	(segment
-		(start 57.92 101.75)
-		(end 79.51 101.75)
-		(width 0.2)
-		(layer "B.Cu")
-		(net 0)
-	)
-	(segment
-		(start 100 57)
-		(end 100 52.1)
+		(start 79.96 102.2)
+		(end 79.96 99.04)
 		(width 0.2)
 		(layer "B.Cu")
@@
 	)
 	(segment
+		(start 36.42 109.42)
+		(end 36.5 109.5)
+		(width 0.2)
+		(layer "B.Cu")
+		(net 0)
+	)
+	(segment
+		(start 57.92 101.75)
+		(end 57.92 109.08)
+		(width 0.2)
+		(layer "B.Cu")
+		(net 0)
+	)
+	(segment
+		(start 79.96 97.54)
+		(end 79.96 102)
+		(width 0.2)
+		(layer "B.Cu")
+		(net 0)
+	)
+	(segment
+		(start 79.96 99.04)
+		(end 81.5 97.5)
+		(width 0.2)
+		(layer "B.Cu")
+		(net 0)
+	)
+	(segment
 		(start 59.42 74)
 		(end 35.42 74)
@@
 	)
 	(segment
+		(start 36.5 109.5)
+		(end 57.5 109.5)
+		(width 0.2)
+		(layer "B.Cu")
+		(net 0)
+	)
+	(segment
+		(start 36.42 101.75)
+		(end 36.42 109.42)
+		(width 0.2)
+		(layer "B.Cu")
+		(net 0)
+	)
+	(segment
 		(start 81.46 73.95)
 		(end 81.46 60.04)
@@
 	)
 	(segment
-		(start 79.96 76.04)
-		(end 80 76)
-		(width 0.2)
-		(layer "B.Cu")
-		(net 0)
-	)
-	(segment
-		(start 81 76)
-		(end 100 57)
-		(width 0.2)
-		(layer "B.Cu")
+		(start 57.5 109.5)
+		(end 57.92 109.08)
+		(width 0.2)
+		(layer "B.Cu")
+		(net 0)
+	)
+	(segment
+		(start 59.5 73.95)
+		(end 59.47 73.95)
+		(width 0.2)
+		(layer "B.Cu")
+		(net 0)
+	)
+	(segment
+		(start 57.92 101.75)
+		(end 57.92 101.5)
+		(width 0.2)
+		(layer "B.Cu")
+		(net 0)
+	)
+	(segment
+		(start 80 97.5)
+		(end 79.96 97.54)
+		(width 0.2)
+		(layer "B.Cu")
+		(net 0)
+	)
+	(segment
+		(start 82.5 96.5)
+		(end 99 96.5)
+		(width 0.2)
+		(layer "B.Cu")
+		(net 0)
+	)
+	(segment
+		(start 79.96 102)
+		(end 79.96 102.2)
+		(width 0.2)
+		(layer "B.Cu")

Commit message: uh
Parts:
- removed the REF** at (40.5, 74.0)
- removed the REF** at (90.5, 47.5)
- removed the REF** at (86.5, 74.0)
- removed the REF** at (73.1, 42.0)
- removed the REF** at (64.5, 74.0)
- removed the REF** at (41.5, 101.8)
- removed the REF** at (63.0, 101.8)
- removed the REF** at (68.0, 42.0)
- removed the REF** at (101.0, 47.5)
- removed the REF** at (60.7, 32.4)
- removed the REF** at (66.8, 51.6)
- removed the REF** at (85.0, 102.2)
- added ?: , , F.Cu at (46.0, 16.0)
- added C1: 22pF, 0603, F.Cu at (21.4, 26.0)
- added C2: 22pF, 0603, F.Cu at (27.5, 26.0)
- added C5: 100nF, 0603, F.Cu at (21.3, 16.2)
- added C6: 100nF, 0603, F.Cu at (30.4, 26.0)
- added D2: , LED-0603, F.Cu at (39.2, 27.4)
- added D3: , LED-0603, F.Cu at (39.2, 29.1)
- added J1: , H3-3.5-11.5X7.0MM, F.Cu at (37.7, 19.9)
- added J2: , H7-2.54, F.Cu at (23.2, 29.2)
- added J3: , H7-2.54, F.Cu at (23.2, 14.0)
- added J4: , H2X3-2.54, F.Cu at (15.8, 21.6)
- added P1: , 2P-SMD-1.78X1.27, B.Cu at (35.1, 21.4)
- added R1: 47k, 0603, F.Cu at (29.4, 16.6)
- added R2: 10k, 0603, F.Cu at (18.1, 16.2)
- added R3: 120R, 0603, F.Cu at (33.0, 26.9)
- added R4: , R0603, F.Cu at (35.9, 27.4)
- added R5: , R0603, F.Cu at (35.9, 29.1)
- added REF**: TO-220-3_Vertical, Package_TO_SOT_THT:TO-220-3_Vertical, F.Cu at (35.9, 35.0)
- added REF**: TO-220-3_Vertical, Package_TO_SOT_THT:TO-220-3_Vertical, F.Cu at (35.9, 42.0)
- added REF**: TO-220-3_Vertical, Package_TO_SOT_THT:TO-220-3_Vertical, F.Cu at (15.0, 34.9)
- added REF**: TO-220-3_Vertical, Package_TO_SOT_THT:TO-220-3_Vertical, F.Cu at (25.4, 35.0)
- added REF**: TO-220-3_Vertical, Package_TO_SOT_THT:TO-220-3_Vertical, F.Cu at (25.4, 42.0)
- added REF**: TO-220-3_Vertical, Package_TO_SOT_THT:TO-220-3_Vertical, F.Cu at (15.0, 41.9)
- added U$3: , LOGO-SEEED-NEW-1X9.6MM, B.Cu at (31.8, 19.2)
- added U1: SN65HVD230, SOIC8-6.0, F.Cu at (30.5, 21.3)
- added U3: MCP2515, TSSOP20-0.65-6.5X4.4MM, F.Cu at (23.3, 20.6)
- added X1: 16MHz, X4-SMD-3.2X2.5X0.7MM, F.Cu at (24.6, 26.0)
Routing:
- net (no net): track 739.6 -> 520.9 mm, vias 8 -> 56
- added copper zone on B.Cu, net (none)
- added copper zone on F.Cu, net (none)
Other:
- board outline added: 28.7 x 18.4 mm
- board text added: "3V"
- board text added: "5V"
- board text added: "Breakout Board"
- board text added: "CAN Bus"
- board text added: "CANH"
- board text added: "CANL"
- board text added: "CS"
- board text added: "D0"
- board text added: "D1"
- board text added: "D10"
- board text added: "D2"
- board text added: "D3"
- board text added: "D4"
- board text added: "D5"
- board text added: "D6"
- board text added: "D7"
- board text added: "D8"
- board text added: "D9"
- board text added: "GND"
- board text added: "P1"
- board text added: "SCK"
- board text added: "SI"
- board text added: "SO"
